File: pc-8033-clone-interface.kicad_sch (KiCad schematic)
At the start: 16 parts, among them J2 80s31, U2 74LS32, U3 74LS04, U4 82C55A, U5 74LS30

Commit message: Some self-doubt comments
Other:
- note added: "The real hardware uses 5.1kΩ but I'm not sure why that would be, and it does not seem to matter. 4.7kΩ is way easier to get"
- note added: "Why does this OR gate exist at all? We could invert ~{IORQ} and gate it into the 74LS30, maybe the timing isn't right"
Changed lines of the file:
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@@
     (stroke (width 0) (type default))
+  )
+  (text "The real hardware uses 5.1kΩ but I'm\nnot sure why that would be, and it\ndoes not seem to matter.\n4.7kΩ is way easier to get"
+    (at 196.85 24.13 0)
+    (effects (font (size 1.27 1.27)) (justify left bottom))
   )
   (text "This second inversion of reset appears to be important for timing purposes,\nas per https://blog.goo.ne.jp/tk-80/e/6ac4226f93ae2f80224ee7fcf31cb796"
@@
     (effects (font (size 1.27 1.27)) (justify left bottom))
   )
+  (text "Why does this OR gate exist at all?\nWe could invert ~{IORQ} and gate it into\nthe 74LS30, maybe the timing isn't right"
+    (at -14.605 81.915 0)
+    (effects (font (size 1.27 1.27)) (justify left bottom))
+  )
